Commit message: fix

File: assets/urdf/arm.urdf (robot description, URDF)
Before this commit: robot arm, 4 links, 3 joints
Links:
- link hand: geometry collision box size=0.06 0.6 0.9; visual box size=0.06 0.6 0.9
- link link1: geometry visual box size=0.06 0.06 0.3
- link link2: geometry visual box size=0.06 0.06 0.3

File: assets/urdf/board_dribble.urdf (robot description, URDF)
Before this commit: robot board, 3 links, 2 joints
Links:
- removed link ball
Joints:
- removed joint slider_to_ball
- joint slider_to_board: limit lower=-4 upper=4 effort=1000.0 velocity=100 -> lower=0 upper=2 effort=1000.0 velocity=100

Commit message: linkの長さを調整

File: assets/urdf/arm.urdf (robot description, URDF)
Before this commit: robot arm, 4 links, 3 joints
Links:
- link link1: geometry visual box size=0.06 0.06 0.6
- link link2: geometry visual box size=0.06 0.06 0.6
Joints:
- joint joint2: origin xyz=0 0 0.3 -> xyz=0 0 0.6
- joint joint3: origin xyz=0 0 0.3 -> xyz=0 0 0.6

Commit message: armをjaxonと同じようにした。maxpusheffortを調整した。関節limitを実装した。ballのz方向の速度0が一定時間続いたらresetをする実装をした。

File: assets/urdf/arm.urdf (robot description, URDF)
Before this commit: robot arm, 4 links, 3 joints
Links:
- link hand: geometry collision box size=0.06 0.2 0.3; visual box size=0.06 0.2 0.3
- link link1: geometry visual box size=0.06 0.06 0.3
- link link2: geometry visual box size=0.06 0.06 0.3
Joints:
- joint joint1: limit lower=-1.0 upper=1.0 effort=200.0 velocity=50 -> lower=-0.75 upper=1.5 effort=200.0 velocity=50
- joint joint2: limit lower=-1.0 upper=1.0 effort=200.0 velocity=50 -> lower=-2.5 upper=0.0 effort=200.0 velocity=50; origin xyz=0 0 0.6 -> xyz=0 0 0.3
- joint joint3: limit lower=-1.0 upper=1.0 effort=200.0 velocity=50 -> lower=-0.75 upper=1.5 effort=200.0 velocity=50; origin xyz=0 0 0.6 -> xyz=0 0 0.3

Commit message: エージェントシステム課題提出

File: assets/urdf/arm.urdf (robot description, URDF)
Before this commit: robot arm, 4 links, 3 joints
Links:
- removed link link1
- removed link link2
- added link elbow-joint-p_link, mass 1; visual cylinder length=0.2 radius=0.02
- added link shoulder-joint-p_link, mass 1; visual cylinder length=0.3 radius=0.02
- added link shoulder-joint-r_link, mass 1; visual cylinder length=0.1 radius=0.02
- added link shoulder-joint-y_link, mass 1; visual cylinder length=0.1 radius=0.02
- added link wrist-joint-r_link, mass 1; visual cylinder length=0.04 radius=0.02
- added link wrist-joint-y_link, mass 1; visual cylinder length=0.1 radius=0.02
- link hand: geometry collision box size=0.3 0.2 0.06; visual box size=0.3 0.2 0.06
Joints:
- removed joint joint1
- removed joint joint2
- removed joint joint3
- added joint elbow-joint-p: type revolute, parent shoulder-joint-p_link, child elbow-joint-p_link, origin xyz=0 0 -0.3 rpy=0 0 0, axis 0 1 0, limit lower=-0.8 upper=1.5708 effort=300.0 velocity=400
- added joint shoulder-joint-p: type revolute, parent shoulder-joint-r_link, child shoulder-joint-p_link, origin xyz=0 -0.04 0, axis 0 1 0, limit lower=-0.5 upper=0.5 effort=300.0 velocity=400
- added joint shoulder-joint-r: type revolute, parent shoulder-joint-y_link, child shoulder-joint-r_link, origin xyz=0 -0.04 0 rpy=0 0 0, axis 1 0 0, limit lower=-0.5 upper=0.0 effort=300.0 velocity=400
- added joint shoulder-joint-y: type revolute, parent base_link, child shoulder-joint-y_link, origin xyz=0 0 0, axis 0 0 1, limit lower=-0.5 upper=0.3 effort=300.0 velocity=400
- added joint wrist-joint-p: type revolute, parent wrist-joint-r_link, child hand, origin xyz=0.02 0 0, axis 0 0 1, limit lower=-0.2 upper=0.2 effort=300.0 velocity=400
- added joint wrist-joint-r: type revolute, parent wrist-joint-y_link, child wrist-joint-r_link, origin xyz=0.12 0 0, axis 0 1 0, limit lower=-1.0 upper=1.5 effort=300.0 velocity=400
- added joint wrist-joint-y: type revolute, parent elbow-joint-p_link, child wrist-joint-y_link, origin xyz=0.2 0 0, axis 1 0 0, limit lower=-0.5 upper=0.5 effort=300.0 velocity=400
